File: tamagotchi.kicad_sch (KiCad schematic)
At the start: 62 parts, among them J1 Conn_01x04_Socket, J2 USB_C_Receptacle_USB2.0_16P, Q1 AO3401A, Q2 2N7002, SW1 SW_SPDT, SW2 SW_Push, SW3 SW_Push, SW4 SW_Push, U1 TP4057-42-SOT26-R, U2 STM32F103C8T6, U3 XC6206P332MR-G, U4 H5VU10BB, U5 H5VU10BB, Y1 16Mhz

Commit message: Hotovo
Parts:
- removed BUZZER1: MLT-5020, easyECADDownloader:BUZ-SMD_L5.0-W5.5-P4.60, symbol easyECADDownloader:MLT-5020
- removed SW2, SW3, SW4: SW_Push, Connector_PinHeader_2.54mm:PinHeader_1x02_P2.54mm_Vertical, symbol Switch:SW_Push
- added BZ1: Buzzer, Connector_PinSocket_2.54mm:PinSocket_1x02_P2.54mm_Vertical, symbol Device:Buzzer
- added C21: 10u, Capacitor_SMD:C_0402_1005Metric, symbol Device:C
- added J3: PAD x4, Connector_PinSocket_2.54mm:PinSocket_1x04_P2.54mm_Vertical, symbol Connector:Conn_01x04_Socket
- added J4: Conn_01x01_Socket, symbol Connector:Conn_01x01_Socket
- added R19: 1k, Resistor_SMD:R_0603_1608Metric, symbol Device:R
- added R20: 5.1k, Resistor_SMD:R_0603_1608Metric, symbol Device:R
- J2: footprint Connector_USB:USB_C_Receptacle_Molex_105450-0101 -> Connector_USB:USB_C_Receptacle_HCTL_HC-TYPE-C-16P-01A
- R1, R5: value 5.1k -> 1k
Connections:
- net +5V: now also D6.2 (A), C21.1; no longer D6.1 (K)
- net +BATT: now also Q1.3 (D); no longer Q1.2 (S)
- net BUT1_SW: now also J3.1 (Pin_1)
- net BUT2_SW: now also J3.2 (Pin_2)
- net BUT3_SW: now also J3.3 (Pin_3)
- net BUZ_DRAIN: now also BZ1.2 (-), R19.2
- net GND: now also C21.2, J3.4 (Pin_4), J4.1 (Pin_1)
- net REG_CHRG: now also D1.1 (K); no longer D2.1 (K)
- net REG_LDO: now also D6.1 (K), Q1.2 (S); no longer D6.2 (A), Q1.3 (D)
- net REG_STBY: now also D2.1 (K); no longer D1.1 (K)
- net USB_D+: now also R20.2
- net VDD: now also BZ1.1 (+), R19.1, R20.1
- net at D2.2 (A): now also R1.1; no longer R5.1
- net at D1.2 (A): now also R5.1; no longer R1.1
- no-connect marks 21 -> 20
Other:
- moved on the sheet: D1, D2, D3, D4, D5, D6, R15, R16, R17, R18, R2, R3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

Commit message: fin
Parts:
- removed C6: 2.2u, Capacitor_SMD:C_0402_1005Metric, symbol Device:C
- removed D6: SS14, Diode_SMD:D_SMA, symbol Diode:SS14
- removed Q2: 2N7002, Package_TO_SOT_SMD:SOT-23, symbol Transistor_FET:2N7002
- removed R19: 1k, Resistor_SMD:R_0603_1608Metric, symbol Device:R
- added C16, C17: 5.6p, Capacitor_SMD:C_0402_1005Metric, symbol Device:C
- added C22: 10u, Capacitor_SMD:C_0603_1608Metric, symbol Device:C
- added D5: RB520S-30, Diode_SMD:D_SOD-523, symbol Device:D_Schottky
- added J1: NRST, Connector_PinHeader_2.54mm:PinHeader_1x01_P2.54mm_Vertical, symbol Connector:Conn_01x01_Socket
- added J6: BAT+, Connector_PinHeader_2.54mm:PinHeader_1x01_P2.54mm_Vertical, symbol Connector:Conn_01x01_Socket
- added Q1: AO3400A, Package_TO_SOT_SMD:SOT-23, symbol Transistor_FET:AO3400A
- added R2, R3, R9: 100k, Resistor_SMD:R_0402_1005Metric, symbol Device:R
- added Y2: 32.768kHz, Crystal:Crystal_SMD_3215-2Pin_3.2x1.5mm, symbol Device:Crystal
- C20: renamed from C21; footprint Capacitor_SMD:C_0402_1005Metric -> Capacitor_SMD:C_0603_1608Metric; LCSC Part C12530 -> C96446
- J2: LCSC C399939 -> C2894897
- J5: renamed from J4; value Conn_01x01_Socket -> BAT-; footprint (none) -> Connector_PinHeader_2.54mm:PinHeader_1x01_P2.54mm_Vertical
- R12: renamed from R2; value 130 -> 150
- R19: renamed from R1; LCSC Part C23186 -> C21190
- R20: renamed from R5; LCSC Part C23186 -> C21190
- R22: renamed from R7; value 2k -> 6.8k; LCSC Part C22975 -> C23212
- R6: renamed from R20; value 5.1k -> 1.5k; footprint Resistor_SMD:R_0603_1608Metric -> Resistor_SMD:R_0402_1005Metric; LCSC Part C23186 -> C25867
- SW1: value SW_SPDT -> SSAJ110100; footprint Button_Switch_SMD:SW_SPST_B3U-1000P -> easyECADDownloader:SW-SMD_SSAJ110100; LCSC Part (none) -> C160863
- renumbered C3 to C1, C16 to C10, C20 to C11, C1 to C12, C2 to C13, C5 to C14, C17 to C15, C4 to C2, C14 to C21, C11 to C23, C7 to C3, C8 to C4, C9 to C5, C10 to C6, C12 to C7, C13 to C8, C15 to C9, D3 to D1, D4 to D2, D5 to D3, D7 to D4, D2 to D6, D1 to D7, J1 to J4, Q1 to Q2, R6 to R1, R15 to R10, R16 to R11, R3 to R13, R4 to R14, R17 to R15, R18 to R16, R10 to R17, R12 to R18, R8 to R21, R13 to R4, R14 to R5, R9 to R7, R11 to R8, U2 to U1, U4 to U2, U5 to U3, U3 to U4, U1 to U5
Connections:
- net +5V: now also D5.2 (A), R2.2
- net +BATT: now also BZ1.1 (+), D4.1 (K), C22.1, J6.1 (Pin_1)
- net BUZ: now also U1.13 (PA3); no longer U1.28 (PB15)
- net BUZ_DRAIN: now also Q1.3 (D)
- net BUZ_GATE: now also Q1.1 (G)
- net DISP_DISP: now also R9.1
- net GND: now also C16.2, C17.2, C22.2, Q1.2 (S), R3.2, R9.2
- net NRST: now also J1.1 (Pin_1)
- net VDD: now also R10.1, R15.1, R4.1; no longer BZ1.1 (+), D4.1 (K), R6.1
- net VDDA: no longer R10.1, R15.1, R4.1
- net at U1.16 (PA6): now also R2.1, R3.1
- net at U1.3 (PC14): now also C16.1, Y2.2
- net at U1.38 (PA15): now also R6.1
- net at U1.4 (PC15): now also C17.1, Y2.1
- net REG_LDO: no longer names the net of C23.1, Q2.2 (S), U4.3 (VI)
- net REG_LDO: now also D5.1 (K)
- no-connect marks 20 -> 16
Other:
- moved on the sheet: C13, C14, D7, J4, R6, Y1

Commit message: abc
Parts:
- U5: footprint Package_TO_SOT_SMD:TSOT-23-6 -> Package_TO_SOT_SMD:SOT-23-6
Changed lines of the file:
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@@
 			)
 		)
-		(property "Footprint" "Package_TO_SOT_SMD:TSOT-23-6"
+		(property "Footprint" "Package_TO_SOT_SMD:SOT-23-6"
 			(at 49.53 190.5 0)
 			(hide yes)
